Commit message: Pruned URDFs and basic node type support for urdfParser

File: urdf_files/A1/a1.urdf (robot description, URDF)
Before this commit: robot a1, 23 links, 22 joints
Links:
- removed link FL_thigh_shoulder
- removed link FR_thigh_shoulder
- removed link RL_thigh_shoulder
- removed link RR_thigh_shoulder
- removed link imu_link
- link FL_calf: mass 0.166 -> 0.151
- link FL_hip: mass 0.696 -> 0.595
- link FL_thigh: mass 1.013 -> 0.888
- link FR_calf: mass 0.166 -> 0.151
- link FR_hip: mass 0.696 -> 0.595
- link FR_thigh: mass 1.013 -> 0.888
- link RL_calf: mass 0.166 -> 0.151
- link RL_hip: mass 0.696 -> 0.595
- link RL_thigh: mass 1.013 -> 0.888
- link RR_calf: mass 0.166 -> 0.151
- link RR_hip: mass 0.696 -> 0.595
- link RR_thigh: mass 1.013 -> 0.888
Joints:
- removed joint FL_hip_fixed
- removed joint FR_hip_fixed
- removed joint RL_hip_fixed
- removed joint RR_hip_fixed
- removed joint imu_joint

File: urdf_files/Go1/go1.urdf (robot description, URDF)
Before this commit: robot go1, 46 links, 45 joints
Links:
- removed link FL_calf_rotor
- removed link FL_hip_rotor
- removed link FL_thigh_rotor
- removed link FR_calf_rotor
- removed link FR_hip_rotor
- removed link FR_thigh_rotor
- removed link RL_calf_rotor
- removed link RL_hip_rotor
- removed link RL_thigh_rotor
- removed link RR_calf_rotor
- removed link RR_hip_rotor
- removed link RR_thigh_rotor
- removed link camera_chin
- removed link camera_face
- removed link camera_laserscan_link_left
- removed link camera_laserscan_link_right
- removed link camera_left
- removed link camera_optical_chin
- removed link camera_optical_face
- removed link camera_optical_left
- removed link camera_optical_rearDown
- removed link camera_optical_right
- removed link camera_rearDown
- removed link camera_right
- removed link imu_link
- removed link ultraSound_face
- removed link ultraSound_left
- removed link ultraSound_right
Joints:
- removed joint FL_calf_rotor_joint
- removed joint FL_hip_rotor_joint
- removed joint FL_thigh_rotor_joint
- removed joint FR_calf_rotor_joint
- removed joint FR_hip_rotor_joint
- removed joint FR_thigh_rotor_joint
- removed joint RL_calf_rotor_joint
- removed joint RL_hip_rotor_joint
- removed joint RL_thigh_rotor_joint
- removed joint RR_calf_rotor_joint
- removed joint RR_hip_rotor_joint
- removed joint RR_thigh_rotor_joint
- removed joint camera_joint_chin
- removed joint camera_joint_face
- removed joint camera_joint_left
- removed joint camera_joint_rearDown
- removed joint camera_joint_right
- removed joint camera_laserscan_joint_left
- removed joint camera_laserscan_joint_right
- removed joint camera_optical_joint_chin
- removed joint camera_optical_joint_face
- removed joint camera_optical_joint_left
- removed joint camera_optical_joint_rearDown
- removed joint camera_optical_joint_right
- removed joint imu_joint
- removed joint ultraSound_joint_face
- removed joint ultraSound_joint_left
- removed joint ultraSound_joint_right

File: urdf_files/HyQ/hyq.urdf (robot description, URDF)
Before this commit: robot hyq, 19 links, 18 joints
Links:
- removed link world
Joints:
- removed joint floating_base_joint
