Commit message: Use Minicheetah urdf to init solo robot graph. Support training with 4 base nodes (but no Morpho-Symm).

File: urdf_files/Solo/solo12.urdf (robot description, URDF)
Before this commit: robot solo, 17 links, 16 joints
Links:
- removed link FL_FOOT
- removed link FL_LOWER_LEG
- removed link FL_SHOULDER
- removed link FL_UPPER_LEG
- removed link FR_FOOT
- removed link FR_LOWER_LEG
- removed link FR_SHOULDER
- removed link FR_UPPER_LEG
- removed link HL_FOOT
- removed link HL_LOWER_LEG
- removed link HL_SHOULDER
- removed link HL_UPPER_LEG
- removed link HR_FOOT
- removed link HR_LOWER_LEG
- removed link HR_SHOULDER
- removed link HR_UPPER_LEG
- added link FL_calf, mass 0.064; collision box size=0.016 0.016 0.2; visual mesh filename=package://yobotics_description/meshes/calf.STL scale=1 1 1
- added link FL_foot, mass 0.15; collision sphere radius=0.025; visual mesh filename=package://yobotics_description/meshes/foot.STL scale=1 1 1
- added link FL_hip, mass 0.57; collision box size=0.09 0.08 0.093; visual mesh filename=package://yobotics_description/meshes/hip.STL scale=1 1 1
- added link FL_thigh, mass 0.634; collision box size=0.043 0.034 0.22; visual mesh filename=package://yobotics_description/meshes/thigh.STL scale=1 1 1
- added link FR_calf, mass 0.064; collision box size=0.016 0.016 0.2; visual mesh filename=package://yobotics_description/meshes/calf.STL scale=1 1 1
- added link FR_foot, mass 0.15; collision sphere radius=0.025; visual mesh filename=package://yobotics_description/meshes/foot.STL scale=1 1 1
- added link FR_hip, mass 0.57; collision box size=0.09 0.08 0.093; visual mesh filename=package://yobotics_description/meshes/hip.STL scale=1 1 1
- added link FR_thigh, mass 0.634; collision box size=0.043 0.034 0.22; visual mesh filename=package://yobotics_description/meshes/thigh.STL scale=1 1 1
- added link RL_calf, mass 0.064; collision box size=0.016 0.016 0.2; visual mesh filename=package://yobotics_description/meshes/calf.STL scale=1 1 1
- added link RL_foot, mass 0.15; collision sphere radius=0.025; visual mesh filename=package://yobotics_description/meshes/foot.STL scale=1 1 1
- added link RL_hip, mass 0.57; collision box size=0.09 0.08 0.093; visual mesh filename=package://yobotics_description/meshes/hip.STL scale=1 1 1
- added link RL_thigh, mass 0.634; collision box size=0.043 0.034 0.22; visual mesh filename=package://yobotics_description/meshes/thigh.STL scale=1 1 1
- added link RR_calf, mass 0.064; collision box size=0.016 0.016 0.2; visual mesh filename=package://yobotics_description/meshes/calf.STL scale=1 1 1
- added link RR_foot, mass 0.15; collision sphere radius=0.025; visual mesh filename=package://yobotics_description/meshes/foot.STL scale=1 1 1
- added link RR_hip, mass 0.57; collision box size=0.09 0.08 0.093; visual mesh filename=package://yobotics_description/meshes/hip.STL scale=1 1 1
- added link RR_thigh, mass 0.634; collision box size=0.043 0.034 0.22; visual mesh filename=package://yobotics_description/meshes/thigh.STL scale=1 1 1
- added link trunk
- link base_link: mass 1.25123725 -> None; geometry visual box size=0.001 0.001 0.001
Joints:
- removed joint FL_ANKLE
- removed joint FL_HAA
- removed joint FL_HFE
- removed joint FL_KFE
- removed joint FR_ANKLE
- removed joint FR_HAA
- removed joint FR_HFE
- removed joint FR_KFE
- removed joint HL_ANKLE
- removed joint HL_HAA
- removed joint HL_HFE
- removed joint HL_KFE
- removed joint HR_ANKLE
- removed joint HR_HAA
- removed joint HR_HFE
- removed joint HR_KFE
- added joint FL_calf_joint: type revolute, parent FL_thigh, child FL_calf, origin xyz=0 0 -0.2115 rpy=0 0 0, axis 0 1 0, limit lower=-3.14159265359 upper=3.14159265359 effort=20 velocity=10.6
- added joint FL_foot_fixed: type fixed, parent FL_calf, child FL_foot, origin xyz=0 0 -0.23039 rpy=0 0 0
- added joint FL_hip_joint: type revolute, parent trunk, child FL_hip, origin xyz=0.196 0.049664 0 rpy=0 0 0, axis 1 0 0, limit lower=-0.872664625997 upper=1.0471975512 effort=20 velocity=10.6
- added joint FL_thigh_joint: type revolute, parent FL_hip, child FL_thigh, origin xyz=0 0.077476 0 rpy=0 0 0, axis 0 1 0, limit lower=-0.523598775598 upper=3.92699081699 effort=20 velocity=10.6
- added joint FR_calf_joint: type revolute, parent FR_thigh, child FR_calf, origin xyz=0 0 -0.2115 rpy=0 0 0, axis 0 1 0, limit lower=-3.14159265359 upper=3.14159265359 effort=20 velocity=10.6
- added joint FR_foot_fixed: type fixed, parent FR_calf, child FR_foot, origin xyz=0 0 -0.23039 rpy=0 0 0
- added joint FR_hip_joint: type revolute, parent trunk, child FR_hip, origin xyz=0.196 -0.049664 0 rpy=0 0 0, axis 1 0 0, limit lower=-1.0471975512 upper=0.872664625997 effort=20 velocity=10.6
- added joint FR_thigh_joint: type revolute, parent FR_hip, child FR_thigh, origin xyz=0 -0.077476 0 rpy=0 0 0, axis 0 1 0, limit lower=-0.523598775598 upper=3.92699081699 effort=20 velocity=10.6
- added joint RL_calf_joint: type revolute, parent RL_thigh, child RL_calf, origin xyz=0 0 -0.2115 rpy=0 0 0, axis 0 1 0, limit lower=-3.14159265359 upper=3.14159265359 effort=20 velocity=10.6
- added joint RL_foot_fixed: type fixed, parent RL_calf, child RL_foot, origin xyz=0 0 -0.23039 rpy=0 0 0
- added joint RL_hip_joint: type revolute, parent trunk, child RL_hip, origin xyz=-0.196 0.049664 0 rpy=0 0 0, axis 1 0 0, limit lower=-0.872664625997 upper=1.0471975512 effort=20 velocity=10.6
- added joint RL_thigh_joint: type revolute, parent RL_hip, child RL_thigh, origin xyz=0 0.077476 0 rpy=0 0 0, axis 0 1 0, limit lower=-0.523598775598 upper=3.92699081699 effort=20 velocity=10.6
- added joint RR_calf_joint: type revolute, parent RR_thigh, child RR_calf, origin xyz=0 0 -0.2115 rpy=0 0 0, axis 0 1 0, limit lower=-3.14159265359 upper=3.14159265359 effort=20 velocity=10.6
- added joint RR_foot_fixed: type fixed, parent RR_calf, child RR_foot, origin xyz=0 0 -0.23039 rpy=0 0 0
- added joint RR_hip_joint: type revolute, parent trunk, child RR_hip, origin xyz=-0.196 -0.049664 0 rpy=0 0 0, axis 1 0 0, limit lower=-1.0471975512 upper=0.872664625997 effort=20 velocity=10.6
- added joint RR_thigh_joint: type revolute, parent RR_hip, child RR_thigh, origin xyz=0 -0.077476 0 rpy=0 0 0, axis 0 1 0, limit lower=-0.523598775598 upper=3.92699081699 effort=20 velocity=10.6
- added joint floating_base: type fixed, parent base_link, child trunk, origin xyz=0 0 0 rpy=0 0 0
